Commit message: added poses

File: hexbot_ws/src/hexbot/urdf/armmove.xacro (robot description, xacro)
@@ -178,4 +178,12 @@
         <box size="0.03 0.03 0.02"/>
       </geometry>
+      <surface>
+        <friction>
+          <ode>
+            <mu>0.1</mu>
+            <mu2>0.1</mu2>
+          </ode>
+        </friction>
+      </surface>
     </collision>
   </link>
@@ -204,4 +212,12 @@
         <box size="0.03 0.03 0.02"/>
       </geometry>
+      <surface>
+        <friction>
+          <ode>
+            <mu>0.1</mu>
+            <mu2>0.1</mu2>
+          </ode>
+        </friction>
+      </surface>
     </collision>
   </link>
@@ -210,5 +226,5 @@
     <parent link="hand"/>
     <child link="fingerright"/>
-    <limit effort="20" lower="0.01" upper="0" velocity="0.2" />
+    <limit effort="20" lower="-0.04" upper="0.0" velocity="0.2" />
   </joint>
 <!--

File: hexbot_ws/src/hexbot/urdf/bot_urdf.xacro (robot description, xacro)
@@ -5,4 +5,6 @@
   <xacro:include filename="$(find hexbot)/urdf/macros.xacro"/>
   <xacro:include filename="$(find hexbot)/urdf/armmove.xacro"/>
+  <xacro:property name="damping_value" value="10" />
+  <xacro:property name="friction_value" value="0.1" />
   <link name="base_footprint">
    <visual>
